File: PCBs/Main Board/ESP32.kicad_sch (KiCad schematic)
At the start: 9 parts, among them SW1 1825910-6, U1 19p_Header, U2 ESP32_WROOM-32U, U3 19p_Header

Commit message: Remove steppers, add OLED
Parts:
- removed SW1: 1825910-6, SnapEDA Library:SW_1825910-6-4, symbol 1825910-6:1825910-6
- added U2: Tactile_Button, Hydro:Tactile_Button, symbol Hydro_Library:Tactile_Button
- added U5: 0.91_OLED, Hydro:0.91 OLED, symbol Hydro_Library:0.91_OLED
- renumbered R6 to R7, U2 to U3, U3 to U4
Connections:
- net 3V3: now also U5.3 (VCC)
- net GND: now also U5.4 (GND)
- net at R7.1: now also U2.3, U2.4
- net at U1.12, U3.12 (19): now also U2.1, U2.2
- net pH_rx renamed SCL
- net SCL: now also U5.2 (SCL)
- net pH_tx renamed SDA
- net SDA: now also U5.1 (SDA)

Commit message: Changed some pins
Parts:
- added D8: LED, LED_THT:LED_D5.0mm, symbol Device:LED
- added R9: R_Small_US, Resistor_THT:R_Axial_DIN0204_L3.6mm_D1.6mm_P7.62mm_Horizontal, symbol Device:R_Small_US
- renumbered R7 to R8
Connections:
- net GND: now also R9.2
- net at U3.24 (13), U4.5: now also D8.2 (A)
- net Part3: now reaches U3.30 (25), U4.11
- net waterLevel: now reaches U3.33 (35), U4.14
- net Nutrients renamed Part1
- net Spare renamed Part2
- new net: D8.1 (K), R9.1
Changed lines of the file:
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@@
   (junction (at 77.47 68.58) (diameter 0) (color 0 0 0 0)
   )
+  (junction (at 77.47 81.28) (diameter 0) (color 0 0 0 0)
+  )
+  (junction (at 77.47 73.66) (diameter 0) (color 0 0 0 0)
+  )
+  (junction (at 77.47 58.42) (diameter 0) (color 0 0 0 0)
+  )
   (wire (pts (xy 48.26 71.12) (xy 50.8 71.12))
     (stroke (width 0) (type default) (color 0 0 0 0))
   )
+  (wire (pts (xy 77.47 58.42) (xy 74.93 58.42))
+    (stroke (width 0) (type default) (color 0 0 0 0))
+  )
   (wire (pts (xy 49.53 78.74) (xy 49.53 93.98))
     (stroke (width 0) (type default) (color 0 0 0 0))
@@
     (stroke (width 0) (type default) (color 0 0 0 0))
   )
-  (wire (pts (xy 77.47 58.42) (xy 74.93 58.42))
+  (wire (pts (xy 87.63 58.42) (xy 77.47 58.42))
     (stroke (width 0) (type default) (color 0 0 0 0))
   )
@@
     (stroke (width 0) (type default) (color 0 0 0 0))
   )
+  (wire (pts (xy 77.47 81.28) (xy 74.93 81.28))
+    (stroke (width 0) (type default) (color 0 0 0 0))
+  )
   (wire (pts (xy 35.56 81.28) (xy 48.26 81.28))
     (stroke (width 0) (type default) (color 0 0 0 0))
@@
     (stroke (width 0) (type default) (color 0 0 0 0))
   )
+  (wire (pts (xy 77.47 73.66) (xy 74.93 73.66))
+    (stroke (width 0) (type default) (color 0 0 0 0))
+  )
   (wire (pts (xy 57.15 120.65) (xy 59.69 120.65))
     (stroke (width 0) (type default) (color 0 0 0 0))
@@
     (stroke (width 0) (type default) (color 0 0 0 0))
   )
-  (wire (pts (xy 77.47 81.28) (xy 74.93 81.28))
-    (stroke (width 0) (type default) (color 0 0 0 0))
-  )
   (wire (pts (xy 48.26 78.74) (xy 49.53 78.74))
     (stroke (width 0) (type default) (color 0 0 0 0))
@@
     (stroke (width 0) (type default) (color 0 0 0 0))
   )
+  (wire (pts (xy 109.22 58.42) (xy 95.25 58.42))
+    (stroke (width 0) (type default) (color 0 0 0 0))
+  )
   (wire (pts (xy 77.47 53.34) (xy 74.93 53.34))
     (stroke (width 0) (type default) (color 0 0 0 0))
@@
     (stroke (width 0) (type default) (color 0 0 0 0))
   )
-  (wire (pts (xy 77.47 73.66) (xy 74.93 73.66))
+  (wire (pts (xy 87.63 73.66) (xy 77.47 73.66))
     (stroke (width 0) (type default) (color 0 0 0 0))
   )
@@
   )
   (wire (pts (xy 34.29 111.76) (xy 105.41 111.76))
+    (stroke (width 0) (type default) (color 0 0 0 0))
+  )
+  (wire (pts (xy 87.63 81.28) (xy 77.47 81.28))
     (stroke (width 0) (type default) (color 0 0 0 0))
   )
@@
     )
   )
-  (global_label "Nutrients" (shape input) (at 39.37 73.66 180) (fields_autoplaced)
+  (global_label "Part1" (shape input) (at 39.37 73.66 180) (fields_autoplaced)
     (effects (font (size 1.27 1.27)) (justify right))
-    (property "Intersheet References" "${INTERSHEET_REFS}" (id 0) (at 28.3693 73.5806 0)
+    (property "Intersheet References" "${INTERSHEET_REFS}" (id 0) (at 31.8164 73.5806 0)
       (effects (font (size 1.27 1.27)) (justify right) hide)
     )
@@
     )
   )
-  (global_label "Spare" (shape input) (at 87.63 68.58 0) (fields_autoplaced)
+  (global_label "Part2" (shape input) (at 87.63 68.58 0) (fields_autoplaced)
     (effects (font (size 1.27 1.27)) (justify left))
-    (property "Intersheet References" "${INTERSHEET_REFS}" (id 0) (at 95.4255 68.5006 0)
+    (property "Intersheet References" "${INTERSHEET_REFS}" (id 0) (at 95.1836 68.5006 0)
+      (effects (font (size 1.27 1.27)) (justify left) hide)
+    )
+  )
+  (global_label "Part3" (shape input) (at 87.63 73.66 0) (fields_autoplaced)
+    (effects (font (size 1.27 1.27)) (justify left))
+    (property "Intersheet References" "${INTERSHEET_REFS}" (id 0) (at 95.1836 73.5806 0)
+      (effects (font (size 1.27 1.27)) (justify left) hide)
+    )
+  )
+  (global_label "waterLevel" (shape input) (at 87.63 81.28 0) (fields_autoplaced)
+    (effects (font (size 1.27 1.27)) (justify left))
+    (property "Intersheet References" "${INTERSHEET_REFS}" (id 0) (at 99.9612 81.2006 0)
       (effects (font (size 1.27 1.27)) (justify left) hide)
     )
@@
   (symbol (lib_id "Device:R_Small_US") (at 59.69 128.27 0) (unit 1)
     (in_bom yes) (on_board yes) (fields_autoplaced)
-    (property "Reference" "R7" (id 0) (at 62.23 126.9999 0)
+    (property "Reference" "R8" (id 0) (at 62.23 126.9999 0)
       (effects (font (size 1.27 1.27)) (justify left))
     )
@@
   (symbol (lib_id "power:GND") (at 59.69 130.81 0) (unit 1)
     (in_bom yes) (on_board yes) (fields_autoplaced)
-    (property "Reference" "#PWR014" (id 0) (at 59.69 137.16 0)
+    (property "Reference" "#PWR016" (id 0) (at 59.69 137.16 0)
       (effects (font (size 1.27 1.27)) hide)
     )
@@
     )
   )
+  (symbol (lib_id "power:GND") (at 109.22 63.5 0) (unit 1)
+    (in_bom yes) (on_board yes) (fields_autoplaced)
+    (property "Reference" "#PWR019" (id 0) (at 109.22 69.85 0)
+      (effects (font (size 1.27 1.27)) hide)
+    )
+    (property "Value" "GND" (id 1) (at 109.22 68.58 0))
+    (property "Footprint" "" (id 2) (at 109.22 63.5 0)
+      (effects (font (size 1.27 1.27)) hide)
+    )
+    (property "Datasheet" "" (id 3) (at 109.22 63.5 0)
+      (effects (font (size 1.27 1.27)) hide)
+    )
+    (pin "1")
+  )
+  (symbol (lib_id "Device:R_Small_US") (at 109.22 60.96 0) (unit 1)
+    (in_bom yes) (on_board yes) (fields_autoplaced)
+    (property "Reference" "R9" (id 0) (at 111.76 59.6899 0)
+      (effects (font (size 1.27 1.27)) (justify left))
+    )
+    (property "Value" "R_Small_US" (id 1) (at 111.76 62.2299 0)
+      (effects (font (size 1.27 1.27)) (justify left))
+    )
+    (property "Footprint" "Resistor_THT:R_Axial_DIN0204_L3.6mm_D1.6mm_P7.62mm_Horizontal" (id 2) (at 109.22 60.96 0)
+      (effects (font (size 1.27 1.27)) hide)
+    )
+    (property "Datasheet" "~" (id 3) (at 109.22 60.96 0)
+      (effects (font (size 1.27 1.27)) hide)
+    )
+    (pin "1")
+    (pin "2")
+  )
+  (symbol (lib_id "Device:LED") (at 91.44 58.42 180) (unit 1)
+    (in_bom yes) (on_board yes) (fields_autoplaced)
+    (property "Reference" "D8" (id 0) (at 93.0275 50.8 0))
+    (property "Value" "LED" (id 1) (at 93.0275 53.34 0))
+    (property "Footprint" "LED_THT:LED_D5.0mm" (id 2) (at 91.44 58.42 0)
+      (effects (font (size 1.27 1.27)) hide)
+    )
+    (property "Datasheet" "~" (id 3) (at 91.44 58.42 0)
+      (effects (font (size 1.27 1.27)) hide)
+    )
+    (pin "1")
+    (pin "2")
+  )
   (symbol (lib_id "Mechanical:MountingHole") (at 156.21 49.53 0) (unit 1)
     (in_bom yes) (on_board yes) (fields_autoplaced)
@@
   (symbol (lib_id "power:GND") (at 90.17 60.96 0) (unit 1)
     (in_bom yes) (on_board yes) (fields_autoplaced)
-    (property "Reference" "#PWR015" (id 0) (at 90.17 67.31 0)
+    (property "Reference" "#PWR017" (id 0) (at 90.17 67.31 0)
       (effects (font (size 1.27 1.27)) hide)
     )
@@
   (symbol (lib_id "power:GND") (at 105.41 116.84 0) (unit 1)
     (in_bom yes) (on_board yes) (fields_autoplaced)
-    (property "Reference" "#PWR016" (id 0) (at 105.41 123.19 0)
+    (property "Reference" "#PWR018" (id 0) (at 105.41 123.19 0)
       (effects (font (size 1.27 1.27)) hide)
     )
@@
   (symbol (lib_id "power:GND") (at 49.53 97.79 0) (unit 1)
     (in_bom yes) (on_board yes) (fields_autoplaced)
-    (property "Reference" "#PWR013" (id 0) (at 49.53 104.14 0)
-      (effects (font (size 1.27 1.27)) hide)
-    )
+    (property "Reference" "#PWR015" (id 0) (at 49.53 104.14 0)
+      (effects (font (size 1.27 1.27)) hide)
+    )
